Commit message: Material "Green" added to avoid warnings

File: create_description/urdf/create_base.urdf.xacro (robot description, xacro)
@@ -2,4 +2,7 @@
 <robot xmlns:xacro="http://ros.org/wiki/xacro">
   <xacro:property name="PI" value="3.1415926535897931" />
+  <material name="Green">
+    <color rgba="0 1 0 1"/>
+  </material>
   <xacro:macro name="create_wheel" params="prefix y_offset wheel_radius wheel_width">
     <link name="${prefix}_wheel_link">
